File: hardware/envelope.kicad_sch (KiCad schematic)
At the start: 63 parts, among them J1 Barrel_Jack_Switch_MountingPin, J2 AudioJack3_Switch, J3 AudioJack3_Switch, SW1 SW_DPDT_x2, SW2 SW_SPDT, U1 4066, U2 4069, U3 4069, U4 4510, U5 CD4052B

Commit message: fix power bug
Parts:
- added C4, C5, C7: 100n, Capacitor_SMD:C_0603_1608Metric_Pad1.08x0.95mm_HandSolder, symbol Device:C
- added D1: D_Schottky, Diode_THT:D_A-405_P7.62mm_Horizontal, symbol Device:D_Schottky
- J2, J3: footprint Connector_Audio:jack_raspi_6.3mmjack -> guitar_stuff:newJack
- RV4: footprint Potentiometer_THT:Potentiometer_TT_P0915N -> guitar_stuff:alpha_poti
- renumbered C7 to C10, C8 to C11, C9 to C12, C10 to C13, C11 to C14, C4 to C6, C5 to C8, C6 to C9, D1 to D2, D2 to D3, TP11 to TP1, TP12 to TP2, TP13 to TP3, TP22 to TP4, TP23 to TP5, TP21 to TP6, TP31 to TP7, TP32 to TP8, TP33 to TP9
Connections:
- net GND: now also J2.R, J2.S, J3.R, J3.S, U2.7 (VSS), U3.7 (VSS), C4.1, C5.1, C7.1; no longer J2.TN, J3.TN, U2.14 (VDD), U3.14 (VDD)
- net VS: now also U2.14 (VDD), U3.14 (VDD), C4.2, C5.2, C7.2; no longer U2.7 (VSS), U3.7 (VSS)
- net at SW1.5 (B): now also J3.T, J3.TN; no longer J3.S
- net at SW1.2 (B): now also J2.T, J2.TN; no longer J2.S
- new net: D1.1 (K), R5.2
- new net: D1.2 (A), J1.2
- now unconnected: J1.3
Other:
- moved on the sheet: J1, TP1, TP4, TP5, TP6, TP7, TP8, U2G, U3G
